File: pcb/bakeneko-65-pcb.kicad_sch (KiCad schematic)
At the start: 18 parts, among them J1 JST SH 4-pin, J2 AVR-ISP-6, SW1 Reset, U1 SRV05-4, U2 ATmega32U4-AU, Y1 16MHz

Commit message: modified:   pcb/bakeneko-65-pcb.kicad_pcb 	modified:   pcb/bakeneko-65-pcb.kicad_prl 	modified:   pcb/bakeneko-65-pcb.kicad_pro 	modified:   pcb/bakeneko-65-pcb.kicad_sch 	modified:   pcb/matrix.kicad_sch 	pcb/Alps_Electric_logo_1960s-1980s.svg 	pcb/random-keyboard-parts.pretty-master/KMULogo.kicad_mod 	pcb/random-keyboard-parts.pretty-master/NeonLogo.kicad_mod
Connections:
- net MISO renamed ENC2B3
Changed lines of the file:
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@@
     (stroke (width 0) (type default))
   )
-  (wire (pts (xy 73.66 92.71) (xy 83.566 92.71))
+  (wire (pts (xy 73.66 92.71) (xy 93.726 92.71))
     (stroke (width 0) (type default))
   )
@@
     (stroke (width 0) (type default))
   )
-  (wire (pts (xy 76.2 97.79) (xy 73.66 97.79))
+  (wire (pts (xy 73.66 97.79) (xy 83.566 97.79))
     (stroke (width 0) (type default))
   )
@@
     )
   )
+  (global_label "ENC2B3" (shape input) (at 83.566 97.79 0) (fields_autoplaced)
+    (effects (font (size 1.27 1.27)) (justify left))
+    (property "Intersheetrefs" "${INTERSHEET_REFS}" (id 0) (at 93.3512 97.79 0)
+      (effects (font (size 1.27 1.27)) (justify left) hide)
+    )
+  )
   (global_label "ROW2" (shape input) (at 76.2 163.83 0)
     (effects (font (size 1.27 1.27)) (justify left))
@@
     (property "Intersheetrefs" "${INTERSHEET_REFS}" (id 0) (at 0 0 0)
       (effects (font (size 1.27 1.27)) hide)
+    )
+  )
+  (global_label "ENC2B1" (shape input) (at 93.726 92.71 0) (fields_autoplaced)
+    (effects (font (size 1.27 1.27)) (justify left))
+    (property "Intersheetrefs" "${INTERSHEET_REFS}" (id 0) (at 103.5112 92.71 0)
+      (effects (font (size 1.27 1.27)) (justify left) hide)
     )
   )
@@
       (reference "#PWR0108") (unit 1) (value "GND") (footprint "")
     )
+    (path "/00000000-0000-0000-0000-00005f45b9b8/decb9a50-ebf1-4bf6-b136-6efaa0d1fa02"
+      (reference "#PWR0109") (unit 1) (value "GND") (footprint "")
+    )
     (path "/00000000-0000-0000-0000-00005f24d3a7"
       (reference "C1") (unit 1) (value "0.1u") (footprint "Capacitor_SMD:C_0805_2012Metric")
@@
       (reference "C9") (unit 1) (value "100nf") (footprint "KeyboardParts:C_0805_2012Metric")
     )
+    (path "/00000000-0000-0000-0000-00005f45b9b8/fc254a1e-32ac-4ee8-ac6b-48cb50599ba3"
+      (reference "C10") (unit 1) (value "100nf") (footprint "KeyboardParts:C_0805_2012Metric")
+    )
+    (path "/00000000-0000-0000-0000-00005f45b9b8/b32c302d-2fa9-4ee3-9d25-4c21ecbfeb2c"
+      (reference "C11") (unit 1) (value "100nf") (footprint "KeyboardParts:C_0805_2012Metric")
+    )
     (path "/00000000-0000-0000-0000-00005f45b9b8/00000000-0000-0000-0000-00005f497530"
       (reference "D1") (unit 1) (value "1N4148") (footprint "KeyboardParts:D_SOD-123-Pretty")
@@
       (reference "ENC1") (unit 1) (value "RotaryEncoder_Switch") (footprint "Rotary_Encoder:RotaryEncoder_Alps_EC11E-Switch_Vertical_H20mm")
     )
+    (path "/00000000-0000-0000-0000-00005f45b9b8/6c07ca53-9324-43dd-a527-2b374a32b055"
+      (reference "ENC2") (unit 1) (value "RotaryEncoder_Switch") (footprint "Rotary_Encoder:RotaryEncoder_Alps_EC11E-Switch_Vertical_H20mm")
+    )
     (path "/00000000-0000-0000-0000-00005f2505eb"
       (reference "F1") (unit 1) (value "500mA") (footprint "Fuse:Fuse_1206_3216Metric")
@@
     )
     (path "/00000000-0000-0000-0000-00005f45b9b8/00000000-0000-0000-0000-00005f497526"
-      (reference "MX2") (unit 1) (value "1u") (footprint "MX_Alps_Hybrid:MX-1U-NoLED")
+      (reference "MX2") (unit 1) (value "1u") (footprint "Alps_Only:ALPS-1U")
     )
     (path "/00000000-0000-0000-0000-00005f45b9b8/00000000-0000-0000-0000-00005f497514"
-      (reference "MX3") (unit 1) (value "1u") (footprint "MX_Alps_Hybrid:MX-1U-NoLED")
+      (reference "MX3") (unit 1) (value "1u") (footprint "Alps_Only:ALPS-1U")
     )
     (path "/00000000-0000-0000-0000-00005f45b9b8/00000000-0000-0000-0000-00005f497502"
-      (reference "MX4") (unit 1) (value "1u") (footprint "MX_Alps_Hybrid:MX-1U-NoLED")
+      (reference "MX4") (unit 1) (value "1u") (footprint "Alps_Only:ALPS-1U")
     )
     (path "/00000000-0000-0000-0000-00005f45b9b8/00000000-0000-0000-0000-00005f49707d"
-      (reference "MX5") (unit 1) (value "1u") (footprint "MX_Alps_Hybrid:MX-1U-NoLED")
+      (reference "MX5") (unit 1) (value "1u") (footprint "Alps_Only:ALPS-1U")
     )
     (path "/00000000-0000-0000-0000-00005f45b9b8/00000000-0000-0000-0000-00005f4974e7"
-      (reference "MX6") (unit 1) (value "1u") (footprint "MX_Alps_Hybrid:MX-1U-NoLED")
+      (reference "MX6") (unit 1) (value "1u") (footprint "Alps_Only:ALPS-1U")
     )
     (path "/00000000-0000-0000-0000-00005f45b9b8/00000000-0000-0000-0000-00005f4974d5"
-      (reference "MX7") (unit 1) (value "1u") (footprint "MX_Alps_Hybrid:MX-1U-NoLED")
+      (reference "MX7") (unit 1) (value "1u") (footprint "Alps_Only:ALPS-1U")
     )
     (path "/00000000-0000-0000-0000-00005f45b9b8/00000000-0000-0000-0000-00005f4974c3"
-      (reference "MX8") (unit 1) (value "1u") (footprint "MX_Alps_Hybrid:MX-1U-NoLED")
+      (reference "MX8") (unit 1) (value "1u") (footprint "Alps_Only:ALPS-1U")
     )
     (path "/00000000-0000-0000-0000-00005f45b9b8/00000000-0000-0000-0000-00005f4974b1"
-      (reference "MX9") (unit 1) (value "1u") (footprint "MX_Alps_Hybrid:MX-1U-NoLED")
+      (reference "MX9") (unit 1) (value "1u") (footprint "Alps_Only:ALPS-1U")
     )
     (path "/00000000-0000-0000-0000-00005f45b9b8/00000000-0000-0000-0000-00005f49749f"
-      (reference "MX10") (unit 1) (value "1u") (footprint "MX_Alps_Hybrid:MX-1U-NoLED")
+      (reference "MX10") (unit 1) (value "1u") (footprint "Alps_Only:ALPS-1U")
     )
     (path "/00000000-0000-0000-0000-00005f45b9b8/00000000-0000-0000-0000-00005f49748d"
-      (reference "MX11") (unit 1) (value "1u") (footprint "MX_Alps_Hybrid:MX-1U-NoLED")
+      (reference "MX11") (unit 1) (value "1u") (footprint "Alps_Only:ALPS-1U")
     )
     (path "/00000000-0000-0000-0000-00005f45b9b8/00000000-0000-0000-0000-00005f49747b"
-      (reference "MX12") (unit 1) (value "1u") (footprint "MX_Alps_Hybrid:MX-1U-NoLED")
+      (reference "MX12") (unit 1) (value "1u") (footprint "Alps_Only:ALPS-1U")
     )
     (path "/00000000-0000-0000-0000-00005f45b9b8/00000000-0000-0000-0000-00005f497469"
-      (reference "MX13") (unit 1) (value "1u") (footprint "MX_Alps_Hybrid:MX-1U-NoLED")
+      (reference "MX13") (unit 1) (value "1u") (footprint "Alps_Only:ALPS-1U")
     )
     (path "/00000000-0000-0000-0000-00005f45b9b8/00000000-0000-0000-0000-00005f497457"
@@
     )
     (path "/00000000-0000-0000-0000-00005f45b9b8/00000000-0000-0000-0000-00005f49733a"
-      (reference "MX32") (unit 1) (value "1u") (footprint "MX_Alps_Hybrid:MX-1U-NoLED")
+      (reference "MX32") (unit 1) (value "1u") (footprint "MX_Only:MXOnly-1U-NoLED")
     )
     (path "/00000000-0000-0000-0000-00005f45b9b8/00000000-0000-0000-0000-00005f4970ab"
@@
       (reference "MX88") (unit 1) (value "2.75u") (footprint "MX_Alps_Hybrid:MX-2.75U-NoLED")
     )
+    (path "/00000000-0000-0000-0000-00005f45b9b8/dd9ca97c-7902-4f93-9a15-fc18666b79eb"
+      (reference "MX89") (unit 1) (value "1.5u") (footprint "MX_Alps_Hybrid:MX-1.5U-NoLED")
+    )
     (path "/00000000-0000-0000-0000-00005f27cfdf"
