File: pcb/matrix.kicad_sch (KiCad schematic)
At the start: 162 parts

Commit message: modified:   pcb/bakeneko-65-pcb.kicad_pcb 	modified:   pcb/matrix.kicad_sch 	modified:   pcb/bakeneko-65-pcb.kicad_sch
Parts:
- added C10, C11: 100nf, KeyboardParts:C_0805_2012Metric, symbol Device:C_Small
- added ENC2: RotaryEncoder_Switch, Rotary_Encoder:RotaryEncoder_Alps_EC11E-Switch_Vertical_H20mm, symbol Device:RotaryEncoder_Switch
- MX32: footprint MX_Alps_Hybrid:MX-1U-NoLED -> MX_Only:MXOnly-1U-NoLED
Connections:
- net COL15: now also ENC2.S2
- net GND: now also C10.2, C11.1, ENC2.C
- net at D31.2 (A), MX32.1 (A): now also ENC2.S1
- new net ENC2B1: C10.1, ENC2.B
- new net ENC2B3: C11.2, ENC2.A
Changed lines of the file:
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@@
   (junction (at 45.72 39.37) (diameter 0) (color 0 0 0 0)
   )
+  (junction (at 265.43 57.15) (diameter 0) (color 0 0 0 0)
+  )
   (junction (at 223.52 100.33) (diameter 0) (color 0 0 0 0)
   )
@@
   (junction (at 237.49 118.11) (diameter 0) (color 0 0 0 0)
   )
+  (junction (at 289.052 58.674) (diameter 0) (color 0 0 0 0)
+  )
   (junction (at 73.66 39.37) (diameter 0) (color 0 0 0 0)
   )
@@
   (junction (at 129.54 132.842) (diameter 0) (color 0 0 0 0)
   )
+  (junction (at 289.052 53.594) (diameter 0) (color 0 0 0 0)
+  )
   (junction (at 223.52 46.99) (diameter 0) (color 0 0 0 0)
   )
@@
   (junction (at 199.39 92.71) (diameter 0) (color 0 0 0 0)
   )
+  (junction (at 289.052 63.754) (diameter 0) (color 0 0 0 0)
+  )
   (junction (at 199.39 74.93) (diameter 0) (color 0 0 0 0)
   )
@@
   (junction (at 255.27 37.846) (diameter 0) (color 0 0 0 0)
   )
+  (junction (at 255.27 56.134) (diameter 0) (color 0 0 0 0)
+  )
   (junction (at 101.6 57.15) (diameter 0) (color 0 0 0 0)
   )
@@
     (stroke (width 0) (type default))
   )
+  (wire (pts (xy 255.27 56.134) (xy 271.018 56.134))
+    (stroke (width 0) (type default))
+  )
   (wire (pts (xy 157.48 57.15) (xy 157.48 39.37))
     (stroke (width 0) (type default))
@@
     (stroke (width 0) (type default))
   )
+  (wire (pts (xy 286.258 58.674) (xy 289.052 58.674))
+    (stroke (width 0) (type default))
+  )
   (wire (pts (xy 166.878 110.49) (xy 168.402 110.49))
     (stroke (width 0) (type default))
@@
     (stroke (width 0) (type default))
   )
+  (wire (pts (xy 269.748 57.15) (xy 265.43 57.15))
+    (stroke (width 0) (type default))
+  )
   (wire (pts (xy 101.6 39.37) (xy 101.6 57.15))
     (stroke (width 0) (type default))
@@
     (stroke (width 0) (type default))
   )
+  (wire (pts (xy 289.052 58.674) (xy 289.306 58.674))
+    (stroke (width 0) (type default))
+  )
   (wire (pts (xy 125.73 82.55) (xy 111.76 82.55))
     (stroke (width 0) (type default))
@@
     (stroke (width 0) (type default))
   )
+  (wire (pts (xy 271.018 61.214) (xy 269.748 61.214))
+    (stroke (width 0) (type default))
+  )
   (wire (pts (xy 59.69 74.93) (xy 59.69 92.71))
     (stroke (width 0) (type default))
@@
     (stroke (width 0) (type default))
   )
+  (wire (pts (xy 255.27 56.134) (xy 255.27 57.15))
+    (stroke (width 0) (type default))
+  )
   (wire (pts (xy 141.478 110.49) (xy 141.478 124.968))
     (stroke (width 0) (type default))
@@
     (stroke (width 0) (type default))
   )
+  (wire (pts (xy 293.116 53.594) (xy 289.052 53.594))
+    (stroke (width 0) (type default))
+  )
   (wire (pts (xy 167.64 64.77) (xy 181.61 64.77))
     (stroke (width 0) (type default))
@@
     (stroke (width 0) (type default))
   )
+  (wire (pts (xy 269.748 61.214) (xy 269.748 57.15))
+    (stroke (width 0) (type default))
+  )
   (wire (pts (xy 195.58 100.33) (xy 209.55 100.33))
     (stroke (width 0) (type default))
@@
     (stroke (width 0) (type default))
   )
+  (wire (pts (xy 286.258 63.754) (xy 286.258 61.214))
+    (stroke (width 0) (type default))
+  )
   (wire (pts (xy 237.49 118.11) (xy 223.52 118.11))
     (stroke (width 0) (type default))
@@
     (stroke (width 0) (type default))
   )
+  (wire (pts (xy 286.258 63.754) (xy 289.052 63.754))
+    (stroke (width 0) (type default))
+  )
   (wire (pts (xy 111.76 82.55) (xy 97.79 82.55))
     (stroke (width 0) (type default))
@@
     (stroke (width 0) (type default))
   )
+  (wire (pts (xy 293.116 63.754) (xy 289.052 63.754))
+    (stroke (width 0) (type default))
+  )
+  (wire (pts (xy 289.052 53.594) (xy 286.258 53.594))
+    (stroke (width 0) (type default))
+  )
   (wire (pts (xy 101.6 74.93) (xy 101.6 92.71))
     (stroke (width 0) (type default))
@@
     (stroke (width 0) (type default))
   )
+  (wire (pts (xy 286.258 53.594) (xy 286.258 56.134))
+    (stroke (width 0) (type default))
+  )
   (wire (pts (xy 143.51 92.71) (xy 143.51 74.93))
     (stroke (width 0) (type default))
@@
     (stroke (width 0) (type default))
   )
-  (wire (pts (xy 255.27 39.37) (xy 255.27 57.15))
+  (wire (pts (xy 255.27 39.37) (xy 255.27 56.134))
     (stroke (width 0) (type default))
   )
@@
     )
   )
+  (global_label "ENC2B3" (shape input) (at 293.116 63.754 0) (fields_autoplaced)
+    (effects (font (size 1.27 1.27)) (justify left))
+    (property "Intersheetrefs" "${INTERSHEET_REFS}" (id 0) (at 302.9012 63.754 0)
+      (effects (font (size 1.27 1.27)) (justify left))
+    )
+  )
   (global_label "COL12" (shape input) (at 213.36 24.13 0)
     (effects (font (size 1.27 1.27)) (justify left))
@@
     )
   )
+  (global_label "ENC2B1" (shape input) (at 293.116 53.594 0) (fields_autoplaced)
+    (effects (font (size 1.27 1.27)) (justify left))
+    (property "Intersheetrefs" "${INTERSHEET_REFS}" (id 0) (at 302.9012 53.594 0)
+      (effects (font (size 1.27 1.27)) (justify left))
+    )
+  )
   (global_label "ENC1B1" (shape input) (at 291.846 35.306 0) (fields_autoplaced)
     (effects (font (size 1.27 1.27)) (justify left))
@@
       (effects (font (size 1.27 1.27)))
     )
-    (property "Footprint" "MX_Alps_Hybrid:MX-1U-NoLED" (id 2) (at 260.35 57.15 0)
+    (property "Footprint" "MX_Only:MXOnly-1U-NoLED" (id 2) (at 260.35 57.15 0)
       (effects (font (size 1.27 1.27)) hide)
     )
@@
     (pin "2")
   )
+  (symbol (lib_id "Device:RotaryEncoder_Switch") (at 278.638 58.674 180) (unit 1)
+    (in_bom yes) (on_board yes) (fields_autoplaced)
+    (property "Reference" "ENC2" (id 0) (at 278.638 50.8 0)
+      (effects (font (size 1.27 1.27)))
+    )
+    (property "Value" "RotaryEncoder_Switch" (id 1) (at 278.638 52.07 0)
+      (effects (font (size 1.27 1.27)))
+    )
+    (property "Footprint" "Rotary_Encoder:RotaryEncoder_Alps_EC11E-Switch_Vertical_H20mm" (id 2) (at 282.448 62.738 0)
+      (effects (font (size 1.27 1.27)) hide)
+    )
+    (property "Datasheet" "~" (id 3) (at 278.638 65.278 0)
+      (effects (font (size 1.27 1.27)) hide)
+    )
+    (pin "A")
+    (pin "B")
+    (pin "C")
+    (pin "S1")
+    (pin "S2")
+  )
   (symbol (lib_id "Switch:SW_SPST") (at 66.548 92.71 0) (mirror y) (unit 1)
     (in_bom yes) (on_board yes)
@@
     (pin "2")
   )
+  (symbol (lib_id "Device:C_Small") (at 289.052 61.214 0) (unit 1)
+    (in_bom yes) (on_board yes) (fields_autoplaced)
+    (property "Reference" "C11" (id 0) (at 292.1 60.5853 0)
+      (effects (font (size 1.27 1.27)) (justify left))
+    )
+    (property "Value" "100nf" (id 1) (at 292.1 61.8553 0)
+      (effects (font (size 1.27 1.27)) (justify left))
+    )
+    (property "Footprint" "KeyboardParts:C_0805_2012Metric" (id 2) (at 289.052 61.214 0)
+      (effects (font (size 1.27 1.27)) hide)
+    )
+    (property "Datasheet" "~" (id 3) (at 289.052 61.214 0)
+      (effects (font (size 1.27 1.27)) hide)
+    )
+    (pin "1")
+    (pin "2")
+  )
   (symbol (lib_id "Device:C_Small") (at 287.782 42.926 0) (unit 1)
     (in_bom yes) (on_board yes) (fields_autoplaced)
@@
     (pin "2")
   )
+  (symbol (lib_id "power:GND") (at 289.306 58.674 90) (unit 1)
+    (in_bom yes) (on_board yes) (fields_autoplaced)
+    (property "Reference" "#PWR0109" (id 0) (at 295.656 58.674 0)
+      (effects (font (size 1.27 1.27)) hide)
+    )
+    (property "Value" "GND" (id 1) (at 293.37 58.674 90)
+      (effects (font (size 1.27 1.27)) (justify right))
+    )
+    (property "Footprint" "" (id 2) (at 289.306 58.674 0)
+      (effects (font (size 1.27 1.27)) hide)
+    )
+    (property "Datasheet" "" (id 3) (at 289.306 58.674 0)
+      (effects (font (size 1.27 1.27)) hide)
+    )
+    (pin "1")
+  )
   (symbol (lib_id "Device:C_Small") (at 287.782 37.846 0) (unit 1)
     (in_bom yes) (on_board yes) (fields_autoplaced)
@@
       (effects (font (size 1.27 1.27)) hide)
     )
+    (pin "1")
+    (pin "2")
+  )
+  (symbol (lib_id "Device:C_Small") (at 289.052 56.134 0) (unit 1)
+    (in_bom yes) (on_board yes) (fields_autoplaced)
+    (property "Reference" "C10" (id 0) (at 292.1 55.5053 0)
+      (effects (font (size 1.27 1.27)) (justify left))
+    )
+    (property "Value" "100nf" (id 1) (at 292.1 56.7753 0)
+      (effects (font (size 1.27 1.27)) (justify left))
+    )
+    (property "Footprint" "KeyboardParts:C_0805_2012Metric" (id 2) (at 289.052 56.134 0)
+      (effects (font (size 1.27 1.27)) hide)
+    )
+    (property "Datasheet" "~" (id 3) (at 289.052 56.134 0)
+      (effects (font (size 1.27 1.27)) hide)
+    )

Commit message: modified:   pcb/bakeneko-65-pcb.kicad_pcb 	modified:   pcb/bakeneko-65-pcb.kicad_prl 	modified:   pcb/bakeneko-65-pcb.kicad_pro 	modified:   pcb/bakeneko-65-pcb.kicad_sch 	modified:   pcb/matrix.kicad_sch 	pcb/Alps_Electric_logo_1960s-1980s.svg 	pcb/random-keyboard-parts.pretty-master/KMULogo.kicad_mod 	pcb/random-keyboard-parts.pretty-master/NeonLogo.kicad_mod
Parts:
- added MX89: 1.5u, MX_Alps_Hybrid:MX-1.5U-NoLED, symbol Switch:SW_SPST
- MX10, MX11, MX12, MX13, MX2, MX3, MX4, MX5, MX6, MX7, MX8, MX9: footprint MX_Alps_Hybrid:MX-1U-NoLED -> Alps_Only:ALPS-1U
Connections:
- net COL0: now also MX89.2 (B)
- net at D32.2 (A), MX33.1 (A), MX34.1 (A): now also MX89.1 (A)
Changed lines of the file:
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@@
   (junction (at 195.58 64.77) (diameter 0) (color 0 0 0 0)
   )
+  (junction (at 41.91 73.66) (diameter 0) (color 0 0 0 0)
+  )
   (junction (at 143.51 57.15) (diameter 0) (color 0 0 0 0)
   )
@@
   (junction (at 227.33 92.71) (diameter 0) (color 0 0 0 0)
   )
+  (junction (at 31.75 77.47) (diameter 0) (color 0 0 0 0)
+  )
   (junction (at 185.42 57.15) (diameter 0) (color 0 0 0 0)
   )
@@
     (stroke (width 0) (type default))
   )
+  (wire (pts (xy 19.558 74.93) (xy 19.558 77.47))
+    (stroke (width 0) (type default))
+  )
   (wire (pts (xy 213.36 92.71) (xy 213.36 110.49))
     (stroke (width 0) (type default))
@@
     (stroke (width 0) (type default))
   )
+  (wire (pts (xy 19.558 77.47) (xy 31.75 77.47))
+    (stroke (width 0) (type default))
+  )
   (wire (pts (xy 241.3 24.13) (xy 241.3 32.512))
     (stroke (width 0) (type default))
@@
     (stroke (width 0) (type default))
   )
+  (wire (pts (xy 29.718 74.93) (xy 29.718 73.66))
+    (stroke (width 0) (type default))
+  )
   (wire (pts (xy 111.76 64.77) (xy 125.73 64.77))
     (stroke (width 0) (type default))
@@
     (stroke (width 0) (type default))
   )
+  (wire (pts (xy 41.91 73.66) (xy 41.91 67.31))
+    (stroke (width 0) (type default))
+  )
   (wire (pts (xy 185.42 74.93) (xy 185.42 92.71))
     (stroke (width 0) (type default))
@@
     (stroke (width 0) (type default))
   )
-  (wire (pts (xy 41.91 74.93) (xy 41.91 67.31))
+  (wire (pts (xy 41.91 74.93) (xy 41.91 73.66))
     (stroke (width 0) (type default))
   )
@@
     (stroke (width 0) (type default))
   )
+  (wire (pts (xy 29.718 73.66) (xy 41.91 73.66))
+    (stroke (width 0) (type default))
+  )
   (wire (pts (xy 181.61 100.33) (xy 195.58 100.33))
     (stroke (width 0) (type default))
@@
       (effects (font (size 1.27 1.27)))
     )
-    (property "Footprint" "MX_Alps_Hybrid:MX-1U-NoLED" (id 2) (at 106.68 39.37 0)
+    (property "Footprint" "Alps_Only:ALPS-1U" (id 2) (at 106.68 39.37 0)
       (effects (font (size 1.27 1.27)) hide)
     )
@@
       (effects (font (size 1.27 1.27)))
     )
-    (property "Footprint" "MX_Alps_Hybrid:MX-1U-NoLED" (id 2) (at 218.44 39.37 0)
+    (property "Footprint" "Alps_Only:ALPS-1U" (id 2) (at 218.44 39.37 0)
       (effects (font (size 1.27 1.27)) hide)
     )
@@
       (effects (font (size 1.27 1.27)))
     )
-    (property "Footprint" "MX_Alps_Hybrid:MX-1U-NoLED" (id 2) (at 204.47 39.37 0)
+    (property "Footprint" "Alps_Only:ALPS-1U" (id 2) (at 204.47 39.37 0)
       (effects (font (size 1.27 1.27)) hide)
     )
@@
       (effects (font (size 1.27 1.27)))
     )
-    (property "Footprint" "MX_Alps_Hybrid:MX-1U-NoLED" (id 2) (at 190.5 39.37 0)
+    (property "Footprint" "Alps_Only:ALPS-1U" (id 2) (at 190.5 39.37 0)
       (effects (font (size 1.27 1.27)) hide)
     )
@@
       (effects (font (size 1.27 1.27)))
     )
-    (property "Footprint" "MX_Alps_Hybrid:MX-1U-NoLED" (id 2) (at 176.53 39.37 0)
+    (property "Footprint" "Alps_Only:ALPS-1U" (id 2) (at 176.53 39.37 0)
       (effects (font (size 1.27 1.27)) hide)
     )
@@
       (effects (font (size 1.27 1.27)))
     )
-    (property "Footprint" "MX_Alps_Hybrid:MX-1U-NoLED" (id 2) (at 162.56 39.37 0)
+    (property "Footprint" "Alps_Only:ALPS-1U" (id 2) (at 162.56 39.37 0)
       (effects (font (size 1.27 1.27)) hide)
     )
@@
       (effects (font (size 1.27 1.27)))
     )
-    (property "Footprint" "MX_Alps_Hybrid:MX-1U-NoLED" (id 2) (at 148.59 39.37 0)
+    (property "Footprint" "Alps_Only:ALPS-1U" (id 2) (at 148.59 39.37 0)
       (effects (font (size 1.27 1.27)) hide)
     )
@@
       (effects (font (size 1.27 1.27)))
     )
-    (property "Footprint" "MX_Alps_Hybrid:MX-1U-NoLED" (id 2) (at 134.62 39.37 0)
+    (property "Footprint" "Alps_Only:ALPS-1U" (id 2) (at 134.62 39.37 0)
       (effects (font (size 1.27 1.27)) hide)
     )
@@
       (effects (font (size 1.27 1.27)))
     )
-    (property "Footprint" "MX_Alps_Hybrid:MX-1U-NoLED" (id 2) (at 120.65 39.37 0)
+    (property "Footprint" "Alps_Only:ALPS-1U" (id 2) (at 120.65 39.37 0)
       (effects (font (size 1.27 1.27)) hide)
     )
@@
       (effects (font (size 1.27 1.27)))
     )
-    (property "Footprint" "MX_Alps_Hybrid:MX-1U-NoLED" (id 2) (at 92.71 39.37 0)
+    (property "Footprint" "Alps_Only:ALPS-1U" (id 2) (at 92.71 39.37 0)
       (effects (font (size 1.27 1.27)) hide)
     )
@@
       (effects (font (size 1.27 1.27)))
     )
-    (property "Footprint" "MX_Alps_Hybrid:MX-1U-NoLED" (id 2) (at 78.74 39.37 0)
+    (property "Footprint" "Alps_Only:ALPS-1U" (id 2) (at 78.74 39.37 0)
       (effects (font (size 1.27 1.27)) hide)
     )
@@
       (effects (font (size 1.27 1.27)))
     )
-    (property "Footprint" "MX_Alps_Hybrid:MX-1U-NoLED" (id 2) (at 64.77 39.37 0)
+    (property "Footprint" "Alps_Only:ALPS-1U" (id 2) (at 64.77 39.37 0)
       (effects (font (size 1.27 1.27)) hide)
     )
@@
       (effects (font (size 1.27 1.27)) hide)
     )
+    (pin "1")
+    (pin "2")
+  )
+  (symbol (lib_id "Switch:SW_SPST") (at 24.638 74.93 0) (mirror y) (unit 1)
+    (in_bom yes) (on_board yes)
+    (property "Reference" "MX89" (id 0) (at 24.638 68.961 0)
+      (effects (font (size 1.27 1.27)))
+    )
+    (property "Value" "1.5u" (id 1) (at 24.638 71.2724 0)
+      (effects (font (size 1.27 1.27)))
+    )
+    (property "Footprint" "MX_Alps_Hybrid:MX-1.5U-NoLED" (id 2) (at 24.638 74.93 0)
+      (effects (font (size 1.27 1.27)) hide)
+    )
+    (property "Datasheet" "~" (id 3) (at 24.638 74.93 0)
+      (effects (font (size 1.27 1.27)) hide)
+    )
